Commit message: refactor(robot): update gripper logic and optimize URDF parsing
- Removed `save_geometry_path` parameter from `gripper()` method.
- Added return types to `Robot` class properties for clarity and type
safety.
- Refactored `_determine_base_link` and `_determine_ee_link` methods for
more robust link determination.
- Introduced improved handling for parallel 2-finger grippers in
`_split_gripper`.
- Removed unused imports and updated debug logging in
`filename_handler_meta`.
- Modified test URDF file handling to dynamically resolve paths and
print additional robot properties.d

This refactor enhances type annotations, improves the gripper logic, and
updates URDF-related functionality.

File: urdf/current.urdf (robot description, URDF)
Before this commit: robot rbs_arm, 14 links, 13 joints
Links:
- link base_link: geometry collision mesh filename=file:///home/narmak/rbs_ws/install/rbs_arm/share/rbs_arm/me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 scale=1.00000 1.00000 1.00000; visual mesh filename=file:///home/narmak/rbs_ws/install/rbs_arm/share/rbs_arm/me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 scale=1.00000 1.00000 1.00000
- link ee_link: geometry collision mesh filename=file:///home/narmak/rbs_ws/install/rbs_arm/share/rbs_arm/me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 scale=1.00000 1.00000 1.00000; visual mesh filename=file:///home/narmak/rbs_ws/install/rbs_arm/share/rbs_arm/me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 scale=1.00000 1.00000 1.00000
- link fork0_link: geometry collision mesh filename=file:///home/narmak/rbs_ws/install/rbs_arm/share/rbs_arm/me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 scale=1.00000 1.00000 1.00000; visual mesh filename=file:///home/narmak/rbs_ws/install/rbs_arm/share/rbs_arm/me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 scale=1.00000 1.00000 1.00000
- link fork1_link: geometry collision mesh filename=file:///home/narmak/rbs_ws/install/rbs_arm/share/rbs_arm/me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 scale=1.00000 1.00000 1.00000; visual mesh filename=file:///home/narmak/rbs_ws/install/rbs_arm/share/rbs_arm/me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 scale=1.00000 1.00000 1.00000
- link fork2_link: geometry collision mesh filename=file:///home/narmak/rbs_ws/install/rbs_arm/share/rbs_arm/me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 scale=1.00000 1.00000 1.00000; visual mesh filename=file:///home/narmak/rbs_ws/install/rbs_arm/share/rbs_arm/me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 scale=1.00000 1.00000 1.00000
- link main0_link: geometry collision mesh filename=file:///home/narmak/rbs_ws/install/rbs_arm/share/rbs_arm/me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 scale=1.00000 1.00000 1.00000; visual mesh filename=file:///home/narmak/rbs_ws/install/rbs_arm/share/rbs_arm/me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 scale=1.00000 1.00000 1.00000
- link main1_link: geometry collision mesh filename=file:///home/narmak/rbs_ws/install/rbs_arm/share/rbs_arm/me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 scale=1.00000 1.00000 1.00000; visual mesh filename=file:///home/narmak/rbs_ws/install/rbs_arm/share/rbs_arm/me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 scale=1.00000 1.00000 1.00000
- link rbs_gripper_gripper_base_link: geometry collision mesh filename=file:///home/narmak/rbs_ws/install/rbs_gripper/share/rbs_gr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; visual mesh filename=file:///home/narmak/rbs_ws/install/rbs_gripper/share/rbs_gr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
- link rbs_gripper_l_finger_link: geometry collision mesh filename=file:///home/narmak/rbs_ws/install/rbs_gripper/share/rbs_gr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; visual mesh filename=file:///home/narmak/rbs_ws/install/rbs_gripper/share/rbs_gr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
- link rbs_gripper_r_finger_link: geometry collision mesh filename=file:///home/narmak/rbs_ws/install/rbs_gripper/share/rbs_gr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; visual mesh filename=file:///home/narmak/rbs_ws/install/rbs_gripper/share/rbs_gr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
- link rbs_gripper_rot_base_link: geometry collision mesh filename=file:///home/narmak/rbs_ws/install/rbs_gripper/share/rbs_gr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; visual mesh filename=file:///home/narmak/rbs_ws/install/rbs_gripper/share/rbs_gr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

File: urdf/test.urdf (robot description, URDF)
Before this commit: robot rbs_arm, 14 links, 1 joints
Links:
- removed link gripper_grasp_point
- removed link rbs_gripper_gripper_base_link
- removed link rbs_gripper_l_finger_link
- removed link rbs_gripper_r_finger_link
- removed link rbs_gripper_rot_base_link
- link base_link: mass 1.88031044620482 -> None; geometry collision mesh filename=/home/narmak/rbs_ws/install/rbs_arm/share/rbs_arm/meshes/co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; visual mesh filename=/home/narmak/rbs_ws/install/rbs_arm/share/rbs_arm/meshes/vi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
- link ee_link: mass 1.88031044620482 -> None; geometry collision mesh filename=/home/narmak/rbs_ws/install/rbs_arm/share/rbs_arm/meshes/co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; visual mesh filename=/home/narmak/rbs_ws/install/rbs_arm/share/rbs_arm/meshes/vi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
- link fork0_link: mass 1.12472202892859 -> None; geometry collision mesh filename=/home/narmak/rbs_ws/install/rbs_arm/share/rbs_arm/meshes/co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; visual mesh filename=/home/narmak/rbs_ws/install/rbs_arm/share/rbs_arm/meshes/vi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
- link fork1_link: mass 1.12472202892859 -> None; geometry collision mesh filename=/home/narmak/rbs_ws/install/rbs_arm/share/rbs_arm/meshes/co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; visual mesh filename=/home/narmak/rbs_ws/install/rbs_arm/share/rbs_arm/meshes/vi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
- link fork2_link: mass 1.12472202892859 -> None; geometry collision mesh filename=/home/narmak/rbs_ws/install/rbs_arm/share/rbs_arm/meshes/co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; visual mesh filename=/home/narmak/rbs_ws/install/rbs_arm/share/rbs_arm/meshes/vi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
- link main0_link: mass 1.58688811563124 -> None; geometry collision mesh filename=/home/narmak/rbs_ws/install/rbs_arm/share/rbs_arm/meshes/co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; visual mesh filename=/home/narmak/rbs_ws/install/rbs_arm/share/rbs_arm/meshes/vi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
- link main1_link: mass 1.58688811563124 -> None; geometry collision mesh filename=/home/narmak/rbs_ws/install/rbs_arm/share/rbs_arm/meshes/co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; visual mesh filename=/home/narmak/rbs_ws/install/rbs_arm/share/rbs_arm/meshes/vi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
