Commit message: refactor(ros2_control): rewrite using jinja2

File: urdf/test.urdf (robot description, URDF)
Before this commit: robot rbs_arm, 9 links, 1 joints
Links:
- added link gripper_grasp_point
- added link rbs_gripper_gripper_base_link, mass None; collision mesh filename=file:///home/narmak/rbs_ws/install/rbs_gripper/share/rbs_gr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; visual mesh filename=file:///home/narmak/rbs_ws/install/rbs_gripper/share/rbs_gr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
- added link rbs_gripper_l_finger_link, mass None; collision mesh filename=file:///home/narmak/rbs_ws/install/rbs_gripper/share/rbs_gr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; visual mesh filename=file:///home/narmak/rbs_ws/install/rbs_gripper/share/rbs_gr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
- added link rbs_gripper_r_finger_link, mass None; collision mesh filename=file:///home/narmak/rbs_ws/install/rbs_gripper/share/rbs_gr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; visual mesh filename=file:///home/narmak/rbs_ws/install/rbs_gripper/share/rbs_gr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
- added link rbs_gripper_rot_base_link, mass None; collision mesh filename=file:///home/narmak/rbs_ws/install/rbs_gripper/share/rbs_gr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; visual mesh filename=file:///home/narmak/rbs_ws/install/rbs_gripper/share/rbs_gr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
- link base_link: geometry collision mesh filename=file:///home/narmak/rbs_ws/install/rbs_arm/share/rbs_arm/me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; visual mesh filename=file:///home/narmak/rbs_ws/install/rbs_arm/share/rbs_arm/me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
- link ee_link: geometry collision mesh filename=file:///home/narmak/rbs_ws/install/rbs_arm/share/rbs_arm/me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; visual mesh filename=file:///home/narmak/rbs_ws/install/rbs_arm/share/rbs_arm/me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
- link fork0_link: geometry collision mesh filename=file:///home/narmak/rbs_ws/install/rbs_arm/share/rbs_arm/me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; visual mesh filename=file:///home/narmak/rbs_ws/install/rbs_arm/share/rbs_arm/me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
- link fork1_link: geometry collision mesh filename=file:///home/narmak/rbs_ws/install/rbs_arm/share/rbs_arm/me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; visual mesh filename=file:///home/narmak/rbs_ws/install/rbs_arm/share/rbs_arm/me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
- link fork2_link: geometry collision mesh filename=file:///home/narmak/rbs_ws/install/rbs_arm/share/rbs_arm/me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; visual mesh filename=file:///home/narmak/rbs_ws/install/rbs_arm/share/rbs_arm/me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
- link main0_link: geometry collision mesh filename=file:///home/narmak/rbs_ws/install/rbs_arm/share/rbs_arm/me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; visual mesh filename=file:///home/narmak/rbs_ws/install/rbs_arm/share/rbs_arm/me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
- link main1_link: geometry collision mesh filename=file:///home/narmak/rbs_ws/install/rbs_arm/share/rbs_arm/me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; visual mesh filename=file:///home/narmak/rbs_ws/install/rbs_arm/share/rbs_arm/me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
